Commit message: fixed the state and command interfaces of the ros2 control xacro

File: ros2/description/urdf/ros2_control.xacro (robot description, xacro)
@@ -28,15 +28,16 @@
                 <state_interface name="velocity"/>
             </joint>
-            <!-- <joint name="LoaderJoint">
-                <command_interface name="position">
-                <param name="min">-1.57</param>
-                <param name="max">1.57</param>
-                </command_interface>
+            <joint name="LoaderJoint">
+                <command_interface name="position"/>
                 <state_interface name="position"/>
                 <state_interface name="velocity"/>
             </joint>
+            <joint name="HopperJoint">
+                <command_interface name="position"/>
+                <state_interface name="position"/>
+            </joint>
             <joint name="DoorJoint">
                 <state_interface name="position"/>
-            </joint> -->
+            </joint>
         </ros2_control>
     </xacro:unless>
@@ -72,7 +73,9 @@
             <joint name="LoaderJoint">
                 <state_interface name="position"/>
+                <command_interface name="position"/>
             </joint>
             <joint name="HopperJoint">
                 <state_interface name="position"/>
+                <command_interface name="position"/>
             </joint>
             <joint name="DoorJoint">
