Commit message: Get lidar in Gazebo working

File: ros2/description/urdf/lidar.xacro (robot description, xacro)
@@ -19,5 +19,34 @@
             </geometry>
         </collision>
-        <!-- IDK how to write inertia values -->
+        <inertial>
+            <origin xyz="0 0 0" rpy="0 0 0"/>
+            <mass value="0.1" />
+            <inertia ixx="${(1/12) * 0.1 * (3*0.05*0.05 + 0.04*0.04)}" ixy="0.0" ixz="0.0"
+                    iyy="${(1/12) * 0.1 * (3*0.05*0.05 + 0.04*0.04)}" iyz="0.0"
+                    izz="${(1/2) * 0.1 * (0.05*0.05)}" />
+        </inertial>
     </link>
+    <gazebo reference="laser_frame">
+        <material>Gazebo/Red</material>
+        <sensor name="laser" type="gpu_lidar">
+            <pose> 0 0 0 0 0 0 </pose>
+            <visualize>true</visualize>
+            <update_rate>10</update_rate>
+            <lidar>
+                <scan>
+                    <horizontal>
+                        <samples>360</samples>
+                        <min_angle>-3.14</min_angle>
+                        <max_angle>3.14</max_angle>
+                    </horizontal>
+                </scan>
+                <range>
+                    <min>0.3</min>
+                    <max>12</max>
+                </range>
+            </lidar>
+            <topic>scan</topic>
+            <gz_frame_id>laser_frame</gz_frame_id>
+        </sensor>
+    </gazebo>
 </robot>

Commit message: Get camera working

File: ros2/description/urdf/lidar.xacro (robot description, xacro)
@@ -5,5 +5,5 @@
         <parent link="Base"/>
         <child link="laser_frame"/>
-        <origin xyz="0 0.3 0" rpy="1.570796 0 0"/>
+        <origin xyz="0 0.3 0" rpy="${pi/2} 0 0"/>
     </joint>
     <link name="laser_frame">

File: ros2/description/urdf/terrence.urdf.xacro (robot description, xacro)
@@ -5,6 +5,8 @@
   <!-- COLORS -->
   <xacro:include filename="colors.xacro"/>
-  <!-- LIDAR TESTING -->
+  <!-- LIDAR -->
   <xacro:include filename="lidar.xacro"/>
+  <!-- CAMERA -->
+  <xacro:include filename="camera.xacro"/>
   <link name="base_link" />
   <link name="base_footprint" />
@@ -62,8 +64,7 @@
     </visual>
     <collision>
-      <origin xyz="-0.030264 6.665E-05 1.2263E-10" rpy="0 0 0" />
-      <geometry>
-        <!-- <mesh filename="file://$(find description)/meshes/DriverWheel.STL" /> -->
-        <sphere radius="0.0397"/>
+      <origin xyz="0 0 0" rpy="0 0 0" />
+      <geometry>
+        <mesh filename="file://$(find description)/meshes/DriverWheel.STL" />
       </geometry>
     </collision>
@@ -79,10 +80,6 @@
   <gazebo reference="DriverWheel">
     <material>Gazebo/Blue</material>
-      <!-- <mu1 value="0.001"/>
-      <mu2 value="0.001"/> -->
       <mu1 value="0.001"/>
       <mu2 value="0.001"/>
-      <!-- <kp value="10000000.0" />
-      <kd value="1.0" /> -->
   </gazebo>
   <link name="DriverSprocket">
@@ -103,8 +100,7 @@
     </visual>
     <collision>
-      <origin xyz="0.0097746 -3.5292E-09 -5.2457E-08" rpy="0 0 0" />
-      <geometry>
-        <!-- <mesh filename="file://$(find description)/meshes/DriverSprocket.STL" /> -->
-        <sphere radius="0.0397"/>
+      <origin xyz="0 0 0" rpy="0 0 0" />
+      <geometry>
+        <mesh filename="file://$(find description)/meshes/DriverSprocket.STL" />
       </geometry>
     </collision>
@@ -119,6 +115,4 @@
   <gazebo reference="DriverSprocket">
     <material>Gazebo/Blue</material>
-      <mu1 value="1.0"/>
-      <mu2 value="1.0"/>
   </gazebo>
   <link name="PassWheel">
@@ -139,8 +133,7 @@
     </visual>
     <collision>
-      <origin xyz="0.020612 8.4006E-05 -0.00023239" rpy="0 0 0" />
-      <geometry>
-        <!-- <mesh filename="file://$(find description)/meshes/PassWheel.STL" /> -->
-        <sphere radius="0.0397"/>
+      <origin xyz="0 0 0" rpy="0 0 0" />
+      <geometry>
+        <mesh filename="file://$(find description)/meshes/PassWheel.STL" />
       </geometry>
     </collision>
@@ -176,8 +169,7 @@
     </visual>
     <collision>
-      <origin xyz="-0.0056813 -3.6211E-09 -5.2434E-08" rpy="0 0 0" />
-      <geometry>
-        <!-- <mesh filename="file://$(find description)/meshes/PassSprocket.STL" /> -->
-        <sphere radius="0.0397"/>
+      <origin xyz="0 0 0" rpy="0 0 0" />
+      <geometry>
+        <mesh filename="file://$(find description)/meshes/PassSprocket.STL" />
       </geometry>
     </collision>
@@ -192,6 +184,4 @@
   <gazebo reference="PassSprocket">
     <material>Gazebo/Blue</material>
-      <mu1 value="1.0"/>
-      <mu2 value="1.0"/>
   </gazebo>
   <link name="Loader">
