Commit message: added colors to terrence parts for distinction

File: ros2/description/urdf/terrence.urdf.xacro (robot description, xacro)
@@ -9,4 +9,8 @@
       <xacro:include filename="gazebo_control.xacro"/>
   </xacro:unless>
+  <!-- COLORS -->
+  <xacro:include filename="colors.xacro"/>
+  <!-- LIDAR TESTING -->
+  <xacro:include filename="lidar.xacro"/>
   <link name="base_link" />
   <link name="base_footprint" />
@@ -28,5 +32,5 @@
         <mesh filename="file://$(find description)/meshes/Base.STL" />
       </geometry>
-      <material name="">
+      <material name="teal">
         <color rgba="0.75294 0.75294 0.75294 1" />
       </material>
@@ -59,5 +63,5 @@
         <mesh filename="file://$(find description)/meshes/DriverWheel.STL" />
       </geometry>
-      <material name="">
+      <material name="green">
         <color rgba="0.79216 0.81961 0.93333 1" />
       </material>
@@ -94,5 +98,5 @@
         <mesh filename="file://$(find description)/meshes/DriverSprocket.STL" />
       </geometry>
-      <material name="">
+      <material name="blue">
         <color rgba="0.79216 0.81961 0.93333 1" />
       </material>
@@ -127,5 +131,5 @@
         <mesh filename="file://$(find description)/meshes/PassWheel.STL" />
       </geometry>
-      <material name="">
+      <material name="purple">
         <color rgba="0.79216 0.81961 0.93333 1" />
       </material>
@@ -162,5 +166,5 @@
         <mesh filename="file://$(find description)/meshes/PassSprocket.STL" />
       </geometry>
-      <material name="">
+      <material name="gray">
         <color rgba="0.79216 0.81961 0.93333 1" />
       </material>
@@ -195,5 +199,5 @@
         <mesh filename="file://$(find description)/meshes/Loader.STL" />
       </geometry>
-      <material name="">
+      <material name="yellow">
         <color rgba="1 0 0 1" />
       </material>
@@ -230,5 +234,5 @@
         <mesh filename="file://$(find description)/meshes/Hopper.STL" />
       </geometry>
-      <material name="">
+      <material name="pink">
         <color rgba="0.79216 0.81961 0.93333 1" />
       </material>
@@ -263,5 +267,5 @@
         <mesh filename="file://$(find description)/meshes/Door.STL" />
       </geometry>
-      <material name="">
+      <material name="silver">
         <color rgba="0.79216 0.81961 0.93333 1" />
       </material>

Commit message: Fix mass value on Base

File: ros2/description/urdf/terrence.urdf.xacro (robot description, xacro)
@@ -19,6 +19,6 @@
   <link name="Base">
     <inertial>
-      <origin xyz="0.0071933 0.035942 -0.37341" rpy="0 0 0" />
-      <mass value="2.0994" />
+     <origin xyz="0.0071933 0.035942 -0.17341" rpy="0 0 0" />
+      <mass value="1.0994" />
       <inertia ixx="0.0052099" ixy="-7.8944E-22" ixz="-4.9264E-20" iyy="0.0060071" iyz="3.293E-21"
         izz="0.0014684" />

Commit message: trying things for auto cycles, not working yet

File: ros2/description/urdf/terrence.urdf.xacro (robot description, xacro)
@@ -358,5 +358,6 @@
     <child link="Door" />
     <axis xyz="1 0 0" />
-    <limit lower="0" upper="0.3927" effort="0" velocity="0" />
+    <limit lower="0" upper="0.3927" effort="0" velocity="5.0" />
+    <dynamics damping="0.05" friction="0.01" />
   </joint>
   <gazebo reference="Door">
